File: main.kicad_sch (KiCad schematic)
At the start: 23 parts, among them J1 Conn_01x02_Socket, U1 ESP32-WROOM-32, U2 LM324

Commit message: make PCB layout
Parts:
- removed C4: C_Small, Capacitor_SMD:C_0504_1310Metric, symbol Device:C_Small
- removed R3: 10R, Resistor_SMD:R_0603_1608Metric, symbol Device:R_Small
- added C1: C_Polarized, Capacitor_SMD:CP_Elec_3x5.3, symbol Device:C_Polarized
- added C5, C6: C_Small, Capacitor_SMD:C_0603_1608Metric, symbol Device:C_Small
Connections:
- net GND: now also C3.2, R1.2, R2.2, R5.1, C1.2, C5.2, C6.2
- net at R7.2, U2.1: now also R11.1; no longer U2.12 (+)
- net at R10.1: now also R20.2; no longer C3.2
- net at R20.1: now also C3.1, R8.1; no longer R18.2
- net at R20.3: now also R9.1; no longer R5.1
- net at R6.2, U2.7: now also R13.1; no longer U2.10 (+)
- new net: C1.1, C5.1, C6.1, R24.1, U2.10 (+), U2.12 (+)
- new net: R18.2, R20.4
Other:
- moved on the sheet: R18, R2, R20, U2E
